File: PCB files/connect4V2.brd (EAGLE design)
At the start: 100 x 60 mm, 58 parts, among them J1 1-2199298-2, U1 PTS526_SK15_SMTR2_LFSSMT_FS-M, U10 WS2813A, U11 WS2813A, U12 WS2813A, U13 WS2813A, U14 WS2813A, U15 WS2813A, U16 WS2813A, U17 WS2813A, U18 WS2813A, U19 WS2813A, U2 PTS526_SK15_SMTR2_LFSSMT_FS-M, U20 WS2813A, U21 WS2813A, U22 WS2813A, U23 WS2813A, U24 WS2813A, U25 WS2813A, U26 WS2813A, U27 WS2813A, U28 WS2813A, U29 WS2813A, U3 PTS526_SK15_SMTR2_LFSSMT_FS-M, U30 WS2813A, U31 WS2813A, U32 WS2813A, U33 WS2813A, U34 WS2813A, U35 WS2813A, U36 WS2813A, U37 WS2813A, U38 WS2813A, U39 WS2813A, U4 PTS526_SK15_SMTR2_LFSSMT_FS-M, U40 WS2813A, U41 WS2813A, U42 WS2813A, U43 WS2813A, U44 WS2813A, U45 WS2813A, U46 WS2813A, U47 WS2813A, U48 PTS526_SK15_SMTR2_LFSSMT_FS-M, U5 WS2813A, U6 WS2813A, U7 WS2813A, U8 WS2813A, U9 WS2813A

Commit message: Add updated EDA files and code with button and LED color change functionality.
Parts:
- R5: value 100K -> 10K
- R7: value 390 -> 330
Changed lines of the file:
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@@
 <attribute name="VALUE" x="43.020940625" y="49.936709375" size="1.27206875" layer="27"/>
 </element>
-<element name="R5" library="Resistor" package="RESAD724W46L381D178B" package3d_urn="urn:adsk.eagle:package:16378561/2" value="100K" x="94.634" y="22" smashed="yes">
+<element name="R5" library="Resistor" package="RESAD724W46L381D178B" package3d_urn="urn:adsk.eagle:package:16378561/2" value="10K" x="94.634" y="22" smashed="yes">
 <attribute name="CATEGORY" value="Resistor" x="94.634" y="22" size="1.778" layer="27" display="off"/>
 <attribute name="MANUFACTURER" value="" x="94.634" y="22" size="1.778" layer="27" display="off"/>
@@
 <attribute name="VENDOR" value="C&amp;K" x="94" y="32" size="1.778" layer="27" display="off"/>
 </element>
-<element name="R7" library="Resistor" package="RESAD724W46L381D178B" package3d_urn="urn:adsk.eagle:package:16378561/2" value="390" x="94.734" y="43" smashed="yes" rot="R270">
+<element name="R7" library="Resistor" package="RESAD724W46L381D178B" package3d_urn="urn:adsk.eagle:package:16378561/2" value="330" x="94.734" y="43" smashed="yes" rot="R270">
 <attribute name="CATEGORY" value="Resistor" x="94.734" y="43" size="1.778" layer="27" rot="R270" display="off"/>
 <attribute name="MANUFACTURER" value="" x="94.734" y="43" size="1.778" layer="27" rot="R270" display="off"/>
