File: PCB files/connect4V2.sch (EAGLE design)
At the start: 58 parts, among them J1 1-2199298-2, U1 PTS526_SK15_SMTR2_LFSSMT_FS-M, U10 WS2813A, U11 WS2813A, U12 WS2813A, U13 WS2813A, U14 WS2813A, U15 WS2813A, U16 WS2813A, U17 WS2813A, U18 WS2813A, U19 WS2813A, U2 PTS526_SK15_SMTR2_LFSSMT_FS-M, U20 WS2813A, U21 WS2813A, U22 WS2813A, U23 WS2813A, U24 WS2813A, U25 WS2813A, U26 WS2813A, U27 WS2813A, U28 WS2813A, U29 WS2813A, U3 PTS526_SK15_SMTR2_LFSSMT_FS-M, U30 WS2813A, U31 WS2813A, U32 WS2813A, U33 WS2813A, U34 WS2813A, U35 WS2813A, U36 WS2813A, U37 WS2813A, U38 WS2813A, U39 WS2813A, U4 PTS526_SK15_SMTR2_LFSSMT_FS-M, U40 WS2813A, U41 WS2813A, U42 WS2813A, U43 WS2813A, U44 WS2813A, U45 WS2813A, U46 WS2813A, U47 WS2813A, U48 PTS526_SK15_SMTR2_LFSSMT_FS-M, U5 WS2813A, U6 WS2813A, U7 WS2813A, U8 WS2813A, U9 WS2813A

Commit message: Add updated EDA files and code with button and LED color change functionality.
Parts:
- R5: value 100K -> 10K
- R7: value 390 -> 330
Changed lines of the file:
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@@
 <part name="U3" library="SMD_Button" library_urn="urn:adsk.wipprod:fs.file:vf.iuqlLaJzROq_oPAzu7-Wkw" deviceset="PTS526_SK15_SMTR2_LFS" device="SMT_FS-M"/>
 <part name="R4" library="Resistor" deviceset="R-US" device="AXIAL-7.2MM-PITCH" package3d_urn="urn:adsk.eagle:package:16378561/2" technology="_" value="10K"/>
-<part name="R5" library="Resistor" deviceset="R-US" device="AXIAL-7.2MM-PITCH" package3d_urn="urn:adsk.eagle:package:16378561/2" technology="_" value="100K"/>
+<part name="R5" library="Resistor" deviceset="R-US" device="AXIAL-7.2MM-PITCH" package3d_urn="urn:adsk.eagle:package:16378561/2" technology="_" value="10K"/>
 <part name="R6" library="Resistor" deviceset="R-US" device="AXIAL-7.2MM-PITCH" package3d_urn="urn:adsk.eagle:package:16378561/2" technology="_" value="470"/>
 <part name="U48" library="SMD_Button" library_urn="urn:adsk.wipprod:fs.file:vf.iuqlLaJzROq_oPAzu7-Wkw" deviceset="PTS526_SK15_SMTR2_LFS" device="SMT_FS-M"/>
-<part name="R7" library="Resistor" deviceset="R-US" device="AXIAL-7.2MM-PITCH" package3d_urn="urn:adsk.eagle:package:16378561/2" technology="_" value="390"/>
+<part name="R7" library="Resistor" deviceset="R-US" device="AXIAL-7.2MM-PITCH" package3d_urn="urn:adsk.eagle:package:16378561/2" technology="_" value="330"/>
 <part name="U$1" library="MICROUSB-5P-FEMALE-AB" library_urn="urn:adsk.wipprod:fs.file:vf.Rhs5KJ4ZRwm7u_a9Xeok_Q" deviceset="MICROUSB-5P-FEMALE-AB" device=""/>
 </parts>
